File: transmitter/breezedude_transmitter.kicad_sch (KiCad schematic)
At the start: 53 parts, among them J1 Conn_01x02_Pin, J11 Conn_01x04_Pin, J2 Conn_01x04_Pin, J3 Conn_01x04_Pin, J4 Conn_01x03_Pin, J5 Conn_01x04_Pin, J6 Conn_01x02_Pin, J7 USB_C_Receptacle_USB2.0_16P, Q2 P-MOS, Q3 P-MOS, SW1 SW_Push, U1 D1213A-04TS-7, U10 D1213A-04TS-7, U2 STLQ015M33R, U3 ATSAMD21G18A-A, U8 HP203B, U9 TP4057

Commit message: V2.5 - some pin changes and improvements. Requires FW 1.2.0+
Parts:
- removed J4: Conn_01x03_Pin, Connector_PinHeader_1.00mm:PinHeader_1x03_P1.00mm_Vertical, symbol Connector:Conn_01x03_Pin
- added C10, C14: 100n 16V, Capacitor_SMD:C_0402_1005Metric, symbol Device:C
- added J8: Conn_01x02_Pin, Connector_PinHeader_1.00mm:PinHeader_1x02_P1.00mm_Vertical, symbol Connector:Conn_01x02_Pin
- added L1: 68nH, Inductor_SMD:L_0603_1608Metric, symbol Device:L
- added R18: 1M5, Resistor_SMD:R_0402_1005Metric, symbol Device:R
- added R19: 4k7, Resistor_SMD:R_0402_1005Metric, symbol Device:R
- added U11: D1213A-04TS-7, footprints:SOT95P280X140-6N, symbol Power_Protection:SRV05-4
- C1: value 47u 6.3V -> 47u 10V; footprint Capacitor_SMD:C_0805_2012Metric -> Capacitor_SMD:C_1206_3216Metric; LCSC C16780 -> C96123
- R13: value 4.7k -> 4k7
- SW1: LCSC C2905184 -> C843674; alt (none) -> C2905184
- U9: LCSC C725791 -> C12044; alt (none) -> C725791
Connections:
- net EN_DCDC is gone; now on net V_DIV: U3.47 (PB02)
- net 3V3: now also C10.2, C14.2, R18.2, U11.5 (VP)
- net ANT: now also L1.2
- net DAVIS_DIR: now also U1.6 (IO4); no longer U1.3 (IO2)
- net DAVIS_SPEED: now also U1.3 (IO2); no longer U1.1 (IO1)
- net GND: now also C10.1, C14.1, L1.1, R19.2, U11.2 (VN)
- net LED2: now also U3.25 (PA16); no longer U3.13 (PA08)
- net LORA_DIO0: no longer U3.25 (PA16)
- net RX: now also U11.6 (IO4); no longer U10.4 (IO3)
- net RX1: now also U11.3 (IO2); no longer U1.4 (IO3)
- net SWDCLK: now also U1.4 (IO3), J8.2 (Pin_2)
- net SWDIO: now also J8.1 (Pin_1)
- net SW_SENSOR: now also R18.1
- net TX: now also U11.4 (IO3); no longer U10.6 (IO4)
- net TX1: now also U11.1 (IO1); no longer U1.6 (IO4)
- net VCC_SENSOR: now also U1.1 (IO1)
- net V_DIV: no longer U3.7 (PB08)
- net HW_Ver1: now reaches U3.39 (PA27)
- net HW_Ver1: now also R19.1
- net HW_Ver2: now reaches U3.41 (PA28)
- new net LED2(alt): U3.13 (PA08)
- new net V_DIV(alt): U3.7 (PB08)
Other:
- moved on the sheet: C6, C7, C8, R13, U10
